File: Gerador de Sinais/Gerador de Sinais.brd (EAGLE design)
At the start: 88.9 x 65.1 mm, 42 parts, among them IC1 TL081P, IC2 TL081P, IC3 TL081P

Commit message: Projetos
Parts:
- moved JP7 67.6 mm to (89.5, 19.7)
- moved JP2 57.4 mm to (84.5, 19.7)
- moved JP3 14.9 mm to (9.53, 59.1)
Routing:
- net -12V: track 197.6 -> 202.1 mm
- net N$5: track 125.6 -> 127.1 mm
- net +12V: track 167.2 -> 166.2 mm
- net GND: track 169.2 -> 168.6 mm
- added copper zone on layer 16, net GND
